Commit message: Add camera and lidar

File: urdf/my_robot.xacro (robot description, xacro)
@@ -6,4 +6,5 @@
     <child link="chassis" />
   </joint>
+  <!--chassis-->
   <link name='chassis'>
     <pose>0 0 0.1 0 0 0</pose>
@@ -54,4 +55,5 @@
     </visual>
   </link>
+  <!--left_wheel-->
   <link name='left_wheel'>
     <pose>0 0 0.1 0 0 0</pose>
@@ -78,4 +80,5 @@
     </visual>
   </link>
+  <!--right_wheel-->
   <link name='right_wheel'>
     <pose>0 0 0.1 0 0 0</pose>
@@ -102,4 +105,5 @@
     </visual>
   </link>
+  <!--Wheel Joints-->
   <joint name="left_wheel_hinge" type="continuous">
     <origin xyz="0 0.15 0" rpy="0 0 0" />
@@ -118,3 +122,72 @@
     <dynamics damping="1.0" friction="1.0"/>
   </joint>
+  <!--camera-->
+  <link name="camera">
+    <collision>
+      <origin xyz="0 0 0" rpy="0 0 0"/>
+      <geometry>
+        <box size="0.05 0.05 0.05"/>
+      </geometry>
+    </collision>
+    <visual>
+      <origin xyz="0 0 0" rpy="0 0 0"/>
+      <geometry>
+        <box size="0.05 0.05 0.05"/>
+      </geometry>
+    </visual>
+    <inertial>
+      <mass value="0.1" />
+      <origin xyz="0 0 0" rpy="0 0 0"/>
+      <inertia ixx="1e-6" ixy="0" ixz="0" iyy="1e-6" iyz="0" izz="1e-6"/>
+      <box_inertia mass="0.1" x="0.05" y="0.05" z="0.05"/>
+    </inertial>
+  </link>
+  <!--camera_joint-->
+  <joint name="camera_joint" type="fixed">
+    <axis xyz="0 1 0" />
+    <origin xyz="0.2 0 0" rpy="0 0 0"/>
+    <parent link="chassis"/>
+    <child link="camera"/>
+  </joint>
+  <!--lidar-->
+  <link name="hokuyo">
+    <collision>
+      <origin xyz="0 0 0" rpy="0 0 0"/>
+      <geometry>
+        <box size="0.1 0.1 0.1"/>
+      </geometry>
+    </collision>
+    <visual>
+      <origin xyz="0 0 0" rpy="0 0 0"/>
+      <geometry filename="package://my_robot/meshes/hokuyo.dae"/>
+    </visual>
+    <inertial>
+      <mass value="1e-5" />
+      <origin xyz="0 0 0" rpy="0 0 0"/>
+      <inertia ixx="1e-6" ixy="0" ixz="0" iyy="1e-6" iyz="0" izz="1e-6" />
+    </inertial>
+  </link>
+  <!--lidar_joint-->
+  <joint name="hokuyo_joint" type="fixed">
+    <axis xyz="0 1 0" />
+    <origin xyz="0.15 0 0.1" rpy="0 0 0"/>
+    <parent link="chassis"/>
+    <child link="hokuyo"/>
+  </joint>
+  <!--add color-->
+  <gazebo reference="left_wheel">
+    <material>Gazebo/Green</material>
+  </gazebo>
+  <gazebo reference="right_wheel">
+    <material>Gazebo/Green</material>
+  </gazebo>
+  <gazebo reference="chassis">
+    <material>Gazebo/Blue</material>
+  </gazebo>
+  <gazebo reference="camera">
+    <material>Gazebo/Black</material>
+  </gazebo>
+  <gazebo reference="hokuyo">
+    <material>Gazebo/Red</material>
+  </gazebo>
 </robot>

Commit message: Update gemometry mesh for lidar

File: urdf/my_robot.xacro (robot description, xacro)
@@ -105,4 +105,61 @@
     </visual>
   </link>
+  <!--camera_joint-->
+  <joint name="camera_joint" type="fixed">
+    <axis xyz="0 1 0" />
+    <origin xyz="0.2 0 0" rpy="0 0 0"/>
+    <parent link="chassis"/>
+    <child link="camera"/>
+  </joint>
+  <!--camera-->
+  <link name="camera">
+    <inertial>
+      <mass value="0.1" />
+      <origin xyz="0 0 0" rpy="0 0 0"/>
+      <inertia ixx="1e-6" ixy="0" ixz="0" iyy="1e-6" iyz="0" izz="1e-6"/>
+    </inertial>
+    <collision name='camera_collision'>
+      <origin xyz="0 0 0" rpy="0 0 0"/>
+      <geometry>
+        <box size="0.05 0.05 0.05"/>
+      </geometry>
+    </collision>
+    <visual name='camera_visual'>
+      <origin xyz="0 0 0" rpy="0 0 0"/>
+      <geometry>
+        <box size="0.05 0.05 0.05"/>
+      </geometry>
+    </visual>
+    <xacro:macro name="box_inertia" mass="0.1" x="0.05" y="0.05" z="0.05">
+      <origin xyz="0 0 0" rpy="0 0 0"/>
+    </xacro:macro>
+  </link>
+  <!--lidar_joint-->
+  <joint name="hokuyo_joint" type="fixed">
+    <axis xyz="0 1 0" />
+    <origin xyz="0.15 0 0.1" rpy="0 0 0"/>
+    <parent link="chassis"/>
+    <child link="hokuyo"/>
+  </joint>
+  <!--lidar-->
+  <link name="hokuyo">
+    <collision name='hokuyo_collision'>
+      <origin xyz="0 0 0" rpy="0 0 0"/>
+      <geometry>
+        <box size="0.1 0.1 0.1"/>
+      </geometry>
+    </collision>
+    <visual name='hokuyo_visual'>
+      <origin xyz="0 0 0" rpy="0 0 0"/>
+      <geometry>
+        <mesh filename="package://my_robot/meshes/hokuyo.dae"/>
+      </geometry>
+    </visual>
+    <inertial>
+      <mass value="1e-5" />
+      <origin xyz="0 0 0" rpy="0 0 0"/>
+      <inertia ixx="1e-6" ixy="0" ixz="0" iyy="1e-6" iyz="0" izz="1e-6" />
+    </inertial>
+  </link>
   <!--Wheel Joints-->
   <joint name="left_wheel_hinge" type="continuous">
@@ -122,57 +179,4 @@
     <dynamics damping="1.0" friction="1.0"/>
   </joint>
-  <!--camera-->
-  <link name="camera">
-    <collision>
-      <origin xyz="0 0 0" rpy="0 0 0"/>
-      <geometry>
-        <box size="0.05 0.05 0.05"/>
-      </geometry>
-    </collision>
-    <visual>
-      <origin xyz="0 0 0" rpy="0 0 0"/>
-      <geometry>
-        <box size="0.05 0.05 0.05"/>
-      </geometry>
-    </visual>
-    <inertial>
-      <mass value="0.1" />
-      <origin xyz="0 0 0" rpy="0 0 0"/>
-      <inertia ixx="1e-6" ixy="0" ixz="0" iyy="1e-6" iyz="0" izz="1e-6"/>
-      <box_inertia mass="0.1" x="0.05" y="0.05" z="0.05"/>
-    </inertial>
-  </link>
-  <!--camera_joint-->
-  <joint name="camera_joint" type="fixed">
-    <axis xyz="0 1 0" />
-    <origin xyz="0.2 0 0" rpy="0 0 0"/>
-    <parent link="chassis"/>
-    <child link="camera"/>
-  </joint>
-  <!--lidar-->
-  <link name="hokuyo">
-    <collision>
-      <origin xyz="0 0 0" rpy="0 0 0"/>
-      <geometry>
-        <box size="0.1 0.1 0.1"/>
-      </geometry>
-    </collision>
-    <visual>
-      <origin xyz="0 0 0" rpy="0 0 0"/>
-      <geometry filename="package://my_robot/meshes/hokuyo.dae"/>
-    </visual>
-    <inertial>
-      <mass value="1e-5" />
-      <origin xyz="0 0 0" rpy="0 0 0"/>
-      <inertia ixx="1e-6" ixy="0" ixz="0" iyy="1e-6" iyz="0" izz="1e-6" />
-    </inertial>
-  </link>
-  <!--lidar_joint-->
-  <joint name="hokuyo_joint" type="fixed">
-    <axis xyz="0 1 0" />
-    <origin xyz="0.15 0 0.1" rpy="0 0 0"/>
-    <parent link="chassis"/>
-    <child link="hokuyo"/>
-  </joint>
   <!--add color-->
   <gazebo reference="left_wheel">
@@ -186,8 +190,8 @@
   </gazebo>
   <gazebo reference="camera">
+    <material>Gazebo/Red</material>
+  </gazebo>
+  <gazebo reference="hokuyo">
     <material>Gazebo/Black</material>
   </gazebo>
-  <gazebo reference="hokuyo">
-    <material>Gazebo/Red</material>
-  </gazebo>
 </robot>
